File: board/mainboard.sch (KiCad schematic (older format))
At the start: 35 parts

Commit message: added power supply circuit
Parts:
- added C?: 10uF/6.3V, ~, symbol C
- added C?: 1nF, ~, symbol C
- added C? (x8): 22uF/6.3V, ~, symbol C
- added C?: 22pF, ~, symbol C
- added C?: 47pF, ~, symbol C
- added C? (x2): 100nF, ~, symbol C
- added C?: 470uF/16V/105C, ~, symbol C
- added D?: 1N5819/SS14, ~, symbol DIODE
- added D?: LED, ~, symbol LED
- added D?: SMBJ6.0, ~, symbol DIODE
- added J?: JACK_2P, ~, symbol JACK_2P
- added L? (x3): 2.2uH/1.5A/DCR<0.1R/CD32, ~, symbol INDUCTOR_SMALL
- added P? (x8): CONN_1, symbol CONN_1
- added Q?: IRF540N, TO220, symbol IRF540N
- added R?: 3.3k/1%, ~, symbol R
- added R?: 4.99k/1%, ~, symbol R
- added R?: 22k/1%, ~, symbol R
- added R?: 100k/1%, ~, symbol R
- added R? (x2): 2.2k, ~, symbol R
- added R?: 51, ~, symbol R
- added R?: 10k(NA), ~, symbol R
- added R?: 1k/1%, ~, symbol R
- added R?: 10k, ~, symbol R
- added SW?: SPST, ~, symbol SPST
- C? (x3): value C -> 22uF/6.3V
- C?: value C -> 22pF
- R?: value R -> Rb
- R?: value R -> Ra
Connections:
- net labels added: +3.3V, +5VP, +5V_OTG_PWR, RESET_N, VAA, VCC, VCOM, VEE
- wire segments 20 -> 169
Other:
- note added: "1.4V_CPU"
- note added: "1.4V_INT"
- note added: "1.5V"
- note added: "3.0VA"
- note added: "POWER SUPPLY"
- moved on the sheet: C?, L?, R?, U?

Commit message: jtag, uart, uext
Parts:
- added R? (x3): 2.2k, ~, symbol R
- added R?: 47k, ~, symbol R
Connections:
- net labels added: PIN37/LED1, SDC0_CMD, SDC0_DATA0, SDC0_DATA1, SDC0_DATA2, SPI2_CLK, SPI2_CS0, SPI2_MISO, SPI2_MOSI, TWI2_SCK, TWI2_SDA, UART1_RX, UART1_TX
- wire segments 169 -> 204
Other:
- note added: "UEXT"

Commit message: updated pdf
Parts:
- added C?: 1nF, ~, symbol C
- added R?: 100k/1%, ~, symbol R
- added R?: 6.8k/1%, ~, symbol R
Connections:
- net labels added: SD0_DATA3, SDC0_SCK, UBOOT
- wire segments 204 -> 160
Other:
- note added: "BUTTON"
- moved on the sheet: D?, P?, R?, SW?
